File: hardware/PDM_1/PDM_1.kicad_pcb (KiCad board)
At the start: 2 copper layers, 60 x 40 mm, 4 parts

Commit message: firmware first update
Parts:
- added C1: 100n, Inductor_SMD:L_0603_1608Metric, F.Cu at (73.5, 98.6)
- added C10: 100n, Capacitor_SMD:C_0603_1608Metric, F.Cu at (62.1, 88.3)
- added C11: 1u, Capacitor_SMD:C_0603_1608Metric, F.Cu at (62.1, 90.8)
- added C12: 10n, Capacitor_SMD:C_0603_1608Metric, F.Cu at (66.1, 78.3)
- added C13: 100n, Capacitor_SMD:C_0603_1608Metric, F.Cu at (66.1, 80.8)
- added C14: 68u, Capacitor_Tantalum_SMD:CP_EIA-7343-31_Kemet-D, F.Cu at (78.8, 88.2)
- added C15: 1u, Capacitor_SMD:C_0603_1608Metric, F.Cu at (66.1, 83.3)
- added C16: 100n, Capacitor_SMD:C_0603_1608Metric, F.Cu at (66.1, 85.8)
- added C17: 100n, Capacitor_SMD:C_0603_1608Metric, F.Cu at (90.4, 71.5)
- added C18: 10uF, Capacitor_SMD:C_0603_1608Metric, F.Cu at (90.4, 74.1)
- added C19: 100n, Capacitor_SMD:C_0603_1608Metric, F.Cu at (90.4, 76.6)
- added C2: 4.7u, Inductor_SMD:L_0603_1608Metric, F.Cu at (73.5, 101.1)
- added C3: 100n, Inductor_SMD:L_0603_1608Metric, F.Cu at (73.5, 103.6)
- added C4: 4.7u, Inductor_SMD:L_0603_1608Metric, F.Cu at (73.5, 106.1)
- added C5: 1u, Capacitor_SMD:C_0603_1608Metric, F.Cu at (62.1, 78.3)
- added C6: 10u, Capacitor_SMD:C_0603_1608Metric, F.Cu at (62.1, 80.8)
- added C7: 100n, Capacitor_SMD:C_0603_1608Metric, F.Cu at (62.1, 83.3)
- added C8: 100n, Capacitor_SMD:C_0603_1608Metric, F.Cu at (62.1, 85.8)
- added C9: 100u, Capacitor_SMD:CP_Elec_6.3x7.7, F.Cu at (154.1, 88.1)
- added D1: 1N5822, Diode_THT:D_DO-201AD_P15.24mm_Horizontal, F.Cu at (62.4, 73.7)
- added D2: D_Zener, Diode_SMD:D_SOD-123, F.Cu at (71.0, 87.0)
- added D3: D_Schottky_Small, Diode_SMD:D_SOD-123, F.Cu at (71.0, 90.3)
- added D4: D_Schottky_Small, Diode_SMD:D_SOD-123, F.Cu at (70.3, 75.4)
- added D5: PESD2CAN.215, Package_TO_SOT_SMD:SOT-23, F.Cu at (99.5, 79.0)
- added FB2: 60R@100MHz, Inductor_SMD:L_0603_1608Metric, F.Cu at (90.4, 79.1)
- added FB3: 60R@100MHz, Inductor_SMD:L_0603_1608Metric, F.Cu at (90.4, 81.6)
- added IC1: BTS722204ESAXUMA1, Samacsys:SOP65P600X115-25N, F.Cu at (92.6, 92.5)
- added IC2: BTS722204ESAXUMA1, Samacsys:SOP65P600X115-25N, F.Cu at (103.1, 92.5)
- added IC3: BTS722204ESAXUMA1, Samacsys:SOP65P600X115-25N, F.Cu at (103.1, 104.8)
- added IC4: BTS722204ESAXUMA1, Samacsys:SOP65P600X115-25N, F.Cu at (92.6, 104.8)
- added IC5: BTS722204ESAXUMA1, Samacsys:SOP65P600X115-25N, F.Cu at (81.7, 102.5)
- added JP1: Jumper_2_Bridged, Connector_PinHeader_2.54mm:PinHeader_1x02_P2.54mm_Vertical, F.Cu at (94.7, 79.1)
- added L1: 300n, Inductor_SMD:L_0603_1608Metric, F.Cu at (66.1, 88.3)
- added R1: 120, Resistor_SMD:R_0603_1608Metric, F.Cu at (90.4, 84.1)
- added U1: STM32G0C1KCTxN, Package_QFP:LQFP-32_7x7mm_P0.8mm, F.Cu at (65.8, 103.0)
- added U2: LD1117S33TR_SOT223, Package_TO_SOT_SMD:SOT-223-3_TabPin2, F.Cu at (73.0, 81.2)
- added U3: LM2675M-5, Package_SO:SOIC-8_3.9x4.9mm_P1.27mm, F.Cu at (135.5, 93.0)
- added U4: ATA6561-GAQW-N, Package_SO:SOIC-8_3.9x4.9mm_P1.27mm, F.Cu at (96.6, 73.5)
Routing:
- added copper zone on F.Cu, net /power/VIN_SW_REG
