File: hardware/PDM_1/PDM_1.kicad_pcb (KiCad board)
At the start: 2 copper layers, 60 x 40 mm, 4 parts

Commit message: Porządki w folderze
Parts:
- added C1: 100n, Inductor_SMD:L_0603_1608Metric, F.Cu at (143.9, 97.7)
- added C10: 100n, Capacitor_SMD:C_0603_1608Metric, F.Cu at (133.1, 73.5)
- added C11: 1u, Capacitor_SMD:C_0603_1608Metric, F.Cu at (138.2, 79.0)
- added C12: 10n, Capacitor_SMD:C_0603_1608Metric, F.Cu at (148.8, 68.9)
- added C13: 100n, Capacitor_SMD:C_0603_1608Metric, F.Cu at (134.6, 82.4)
- added C14: 68u, Capacitor_SMD:CP_Elec_6.3x5.4, F.Cu at (137.6, 66.2)
- added C15: 1u, Capacitor_SMD:C_0603_1608Metric, F.Cu at (142.5, 72.2)
- added C16: 100n, Capacitor_SMD:C_0603_1608Metric, F.Cu at (142.5, 70.7)
- added C17: 100n, Capacitor_SMD:C_0603_1608Metric, F.Cu at (134.4, 125.0)
- added C18: 10uF, Capacitor_SMD:C_0603_1608Metric, F.Cu at (136.0, 120.4)
- added C19: 100n, Capacitor_SMD:C_0603_1608Metric, F.Cu at (136.1, 118.9)
- added C2: 4.7u, Inductor_SMD:L_0603_1608Metric, F.Cu at (142.4, 97.7)
- added C29: 220p, Capacitor_SMD:C_0603_1608Metric_Pad1.08x0.95mm_HandSolder, F.Cu at (154.7, 156.1)
- added C3: 100n, Inductor_SMD:L_0603_1608Metric, F.Cu at (129.7, 94.7)
- added C30: 100n, Capacitor_SMD:C_0603_1608Metric_Pad1.08x0.95mm_HandSolder, F.Cu at (153.2, 141.3)
- added C31: 22n, Capacitor_SMD:C_0603_1608Metric_Pad1.08x0.95mm_HandSolder, F.Cu at (158.6, 142.5)
- added C32: 470n, Capacitor_SMD:C_0603_1608Metric_Pad1.08x0.95mm_HandSolder, F.Cu at (155.7, 143.7)
- added C33: 10n, Capacitor_SMD:C_0603_1608Metric_Pad1.08x0.95mm_HandSolder, B.Cu at (171.5, 141.5)
- added C34: 10n, Capacitor_SMD:C_0603_1608Metric_Pad1.08x0.95mm_HandSolder, B.Cu at (171.5, 145.3)
- added C35: 10n, Capacitor_SMD:C_0603_1608Metric_Pad1.08x0.95mm_HandSolder, B.Cu at (171.5, 149.2)
- added C37: 220p, Capacitor_SMD:C_0603_1608Metric_Pad1.08x0.95mm_HandSolder, F.Cu at (154.7, 136.1)
- added C38: 100n, Capacitor_SMD:C_0603_1608Metric_Pad1.08x0.95mm_HandSolder, F.Cu at (155.2, 121.2)
- added C39: 22n, Capacitor_SMD:C_0603_1608Metric_Pad1.08x0.95mm_HandSolder, F.Cu at (158.6, 122.5)
- added C4: 4.7u, Inductor_SMD:L_0603_1608Metric, F.Cu at (129.7, 96.2)
- added C40: 470n, Capacitor_SMD:C_0603_1608Metric_Pad1.08x0.95mm_HandSolder, F.Cu at (155.7, 123.7)
- added C41: 10n, Capacitor_SMD:C_0603_1608Metric_Pad1.08x0.95mm_HandSolder, B.Cu at (171.5, 126.2)
- added C42: 10n, Capacitor_SMD:C_0603_1608Metric_Pad1.08x0.95mm_HandSolder, B.Cu at (171.5, 130.0)
- added C43: 10n, Capacitor_SMD:C_0603_1608Metric_Pad1.08x0.95mm_HandSolder, B.Cu at (171.5, 133.9)
- added C44: 10n, Capacitor_SMD:C_0603_1608Metric_Pad1.08x0.95mm_HandSolder, B.Cu at (171.5, 137.7)
- added C45: 220p, Capacitor_SMD:C_0603_1608Metric_Pad1.08x0.95mm_HandSolder, F.Cu at (154.7, 116.1)
- added C46: 100n, Capacitor_SMD:C_0603_1608Metric_Pad1.08x0.95mm_HandSolder, F.Cu at (153.2, 101.3)
- added C47: 22n, Capacitor_SMD:C_0603_1608Metric_Pad1.08x0.95mm_HandSolder, F.Cu at (158.6, 102.5)
- added C48: 470n, Capacitor_SMD:C_0603_1608Metric_Pad1.08x0.95mm_HandSolder, F.Cu at (155.7, 103.7)
- added C49: 10n, Capacitor_SMD:C_0603_1608Metric_Pad1.08x0.95mm_HandSolder, B.Cu at (171.5, 100.4)
- added C5: 1u, Capacitor_SMD:C_0603_1608Metric, F.Cu at (159.4, 74.8)
- added C50: 10n, Capacitor_SMD:C_0603_1608Metric_Pad1.08x0.95mm_HandSolder, B.Cu at (171.5, 104.2)
- added C51: 10n, Capacitor_SMD:C_0603_1608Metric_Pad1.08x0.95mm_HandSolder, B.Cu at (171.5, 108.0)
- added C52: 10n, Capacitor_SMD:C_0603_1608Metric_Pad1.08x0.95mm_HandSolder, B.Cu at (171.5, 111.9)
- added C53: 220p, Capacitor_SMD:C_0603_1608Metric_Pad1.08x0.95mm_HandSolder, F.Cu at (154.7, 96.0)
- added C54: 100n, Capacitor_SMD:C_0603_1608Metric_Pad1.08x0.95mm_HandSolder, F.Cu at (153.2, 81.2)
- added C55: 22n, Capacitor_SMD:C_0603_1608Metric_Pad1.08x0.95mm_HandSolder, F.Cu at (158.6, 82.4)
- added C56: 470n, Capacitor_SMD:C_0603_1608Metric_Pad1.08x0.95mm_HandSolder, F.Cu at (155.7, 83.6)
- added C57: 10n, Capacitor_SMD:C_0603_1608Metric_Pad1.08x0.95mm_HandSolder, B.Cu at (171.5, 85.2)
- added C58: 10n, Capacitor_SMD:C_0603_1608Metric_Pad1.08x0.95mm_HandSolder, B.Cu at (171.5, 89.0)
- added C59: 10n, Capacitor_SMD:C_0603_1608Metric_Pad1.08x0.95mm_HandSolder, B.Cu at (171.5, 92.8)
- added C6: 10u, Capacitor_SMD:C_0603_1608Metric, F.Cu at (157.9, 74.8)
- added C60: 10n, Capacitor_SMD:C_0603_1608Metric_Pad1.08x0.95mm_HandSolder, B.Cu at (171.5, 96.6)
- added C7: 100n, Capacitor_SMD:C_0603_1608Metric, F.Cu at (156.4, 74.8)
- added C8: 100n, Capacitor_SMD:C_0603_1608Metric, F.Cu at (154.9, 74.8)
- added C9: 100u, Capacitor_SMD:CP_Elec_6.3x7.7, F.Cu at (156.7, 66.1)
- added D1: LED, LED_SMD:LED_0603_1608Metric, F.Cu at (137.8, 150.3)
- added D10: D_Schottky, Diode_SMD:D_SMA, F.Cu at (160.6, 116.2)
- added D11: D_Schottky, Diode_SMD:D_SMA, F.Cu at (160.6, 96.1)
- added D2: LED, LED_SMD:LED_0603_1608Metric, F.Cu at (137.8, 153.4)
- added D3: PESD24VF1BLYL, Diode_SMD:D_SMA, F.Cu at (162.2, 66.1)
- added D3: D_Schottky_Small, Diode_SMD:D_SOD-123, F.Cu at (161.4, 75.8)
- added D4: D_Schottky_Small, Diode_SMD:D_SOD-123, F.Cu at (151.6, 63.5)
- added D5: PESD2CAN.215, Package_TO_SOT_SMD:SOT-23, F.Cu at (137.2, 135.9)
- added D7: LED, LED_SMD:LED_0603_1608Metric, F.Cu at (137.8, 156.6)
- added D8: D_Schottky, Diode_SMD:D_SMA, F.Cu at (160.6, 156.2)
- added D9: D_Schottky, Diode_SMD:D_SMA, F.Cu at (160.6, 136.2)
- added Dr1: SS34ALH, Diode_SMD:D_SMA, F.Cu at (163.7, 71.6)
- added F1: 2920L050_72DR, 2920l:FUSC7451X125N, F.Cu at (168.5, 76.4)
- added FB1: FerriteBead_Small, Inductor_SMD:L_0603_1608Metric, F.Cu at (129.7, 93.2)
- added FB2: 60R@100MHz, Inductor_SMD:L_0603_1608Metric, F.Cu at (132.9, 125.0)
- added FB3: 60R@100MHz, Inductor_SMD:L_0603_1608Metric, F.Cu at (139.0, 120.4)
- added IC2: BTS722204ESAXUMA1, Samacsys:SOP65P600X115-25N, F.Cu at (160.4, 148.2)
- added IC3: BTS722204ESAXUMA1, Samacsys:SOP65P600X115-25N, F.Cu at (160.4, 128.2)
- added IC4: BTS722204ESAXUMA1, Samacsys:SOP65P600X115-25N, F.Cu at (160.4, 108.2)
- added IC5: BTS722204ESAXUMA1, Samacsys:SOP65P600X115-25N, F.Cu at (160.4, 88.1)
- added J1: FTSH-107-01-L-DV-K-A, FTSH-107-01-L-DV-K-A:FTSH-107-XX-YYY-DV-K-A, F.Cu at (135.4, 112.1)
- added J2: UPT-08-01-01-L-RA, proper_8pin:UPT080101LRA, F.Cu at (178.9, 112.9)
- added J5: UPT-02-01-01-X-RA, 2pin:SAMTEC_UPT-02-01-01-X-RA, F.Cu at (177.4, 68.9)
- added J6: Conn_01x06, Connector_IDC:IDC-Header_2x03_P2.54mm_Vertical, F.Cu at (128.4, 139.8)
- added J7: UPT-08-01-01-L-RA, proper_8pin:UPT080101LRA, F.Cu at (178.9, 154.0)
- added JP1: Jumper_2_Bridged, Connector_PinHeader_2.54mm:PinHeader_1x02_P2.54mm_Vertical, F.Cu at (139.7, 128.6)
- added L1: 300n, Inductor_SMD:L_0603_1608Metric, F.Cu at (157.2, 72.5)
- added L4: 47u, Inductor_SMD:L_6.3x6.3_H3, F.Cu at (146.0, 64.6)
- added R1: 120, Resistor_SMD:R_0603_1608Metric, F.Cu at (134.3, 128.5)
- added R10: 1.2k, Resistor_SMD:R_0603_1608Metric, F.Cu at (147.2, 104.5)
- added R11: 4.7k, Resistor_SMD:R_0603_1608Metric_Pad0.98x0.95mm_HandSolder, F.Cu at (156.2, 156.1)
- added R12: 470, Resistor_SMD:R_0603_1608Metric_Pad0.98x0.95mm_HandSolder, F.Cu at (153.2, 144.3)
- added R13: 4.7k, Resistor_SMD:R_0603_1608Metric_Pad0.98x0.95mm_HandSolder, F.Cu at (157.8, 153.6)
- added R14: 10k, Resistor_SMD:R_0603_1608Metric_Pad0.98x0.95mm_HandSolder, F.Cu at (150.5, 152.8)
- added R15: 10k, Resistor_SMD:R_0603_1608Metric_Pad0.98x0.95mm_HandSolder, F.Cu at (152.0, 152.8)
- added R16: 10k, Resistor_SMD:R_0603_1608Metric_Pad0.98x0.95mm_HandSolder, F.Cu at (153.5, 152.8)
- added R17: 10k, Resistor_SMD:R_0603_1608Metric_Pad0.98x0.95mm_HandSolder, F.Cu at (155.0, 152.8)
- added R18: 47, Resistor_SMD:R_0603_1608Metric_Pad0.98x0.95mm_HandSolder, F.Cu at (153.2, 142.8)
- added R19: 1.2k, Resistor_SMD:R_0603_1608Metric_Pad0.98x0.95mm_HandSolder, F.Cu at (161.1, 153.6)
- added R2: 1.2k, Resistor_SMD:R_0603_1608Metric, F.Cu at (147.2, 144.5)
- added R20: 4.7k, Resistor_SMD:R_0603_1608Metric_Pad0.98x0.95mm_HandSolder, F.Cu at (156.2, 136.1)
- added R21: 470, Resistor_SMD:R_0603_1608Metric_Pad0.98x0.95mm_HandSolder, F.Cu at (153.2, 124.3)
- added R22: 4.7k, Resistor_SMD:R_0603_1608Metric_Pad0.98x0.95mm_HandSolder, F.Cu at (157.8, 133.6)
- added R23: 10k, Resistor_SMD:R_0603_1608Metric_Pad0.98x0.95mm_HandSolder, F.Cu at (150.5, 132.8)
- added R24: 10k, Resistor_SMD:R_0603_1608Metric_Pad0.98x0.95mm_HandSolder, F.Cu at (152.0, 132.8)
- added R25: 10k, Resistor_SMD:R_0603_1608Metric_Pad0.98x0.95mm_HandSolder, F.Cu at (153.5, 132.8)
- added R26: 10k, Resistor_SMD:R_0603_1608Metric_Pad0.98x0.95mm_HandSolder, F.Cu at (155.0, 132.8)
- added R27: 47, Resistor_SMD:R_0603_1608Metric_Pad0.98x0.95mm_HandSolder, F.Cu at (153.2, 122.8)
- added R28: 1.2k, Resistor_SMD:R_0603_1608Metric_Pad0.98x0.95mm_HandSolder, F.Cu at (161.1, 133.6)
- added R29: 4.7k, Resistor_SMD:R_0603_1608Metric_Pad0.98x0.95mm_HandSolder, F.Cu at (156.2, 116.1)
- added R3: 1.2k, Resistor_SMD:R_0603_1608Metric, F.Cu at (147.2, 146.0)
- added R30: 470, Resistor_SMD:R_0603_1608Metric_Pad0.98x0.95mm_HandSolder, F.Cu at (153.2, 104.3)
- added R31: 4.7k, Resistor_SMD:R_0603_1608Metric_Pad0.98x0.95mm_HandSolder, F.Cu at (157.8, 113.6)
- added R32: 10k, Resistor_SMD:R_0603_1608Metric_Pad0.98x0.95mm_HandSolder, F.Cu at (150.5, 112.8)
- added R33: 10k, Resistor_SMD:R_0603_1608Metric_Pad0.98x0.95mm_HandSolder, F.Cu at (152.0, 112.8)
- added R34: 10k, Resistor_SMD:R_0603_1608Metric_Pad0.98x0.95mm_HandSolder, F.Cu at (153.5, 112.8)
- added R35: 10k, Resistor_SMD:R_0603_1608Metric_Pad0.98x0.95mm_HandSolder, F.Cu at (155.0, 112.8)
- added R36: 47, Resistor_SMD:R_0603_1608Metric_Pad0.98x0.95mm_HandSolder, F.Cu at (153.2, 102.8)
- added R37: 1.2k, Resistor_SMD:R_0603_1608Metric_Pad0.98x0.95mm_HandSolder, F.Cu at (161.1, 113.6)
- added R38: 4.7k, Resistor_SMD:R_0603_1608Metric_Pad0.98x0.95mm_HandSolder, F.Cu at (156.2, 96.0)
- added R39: 470, Resistor_SMD:R_0603_1608Metric_Pad0.98x0.95mm_HandSolder, F.Cu at (153.2, 84.2)
- added R4: 1.2k, Resistor_SMD:R_0603_1608Metric, F.Cu at (147.2, 147.5)
- added R40: 4.7k, Resistor_SMD:R_0603_1608Metric_Pad0.98x0.95mm_HandSolder, F.Cu at (157.8, 93.5)
- added R41: 10k, Resistor_SMD:R_0603_1608Metric_Pad0.98x0.95mm_HandSolder, F.Cu at (150.5, 92.7)
- added R42: 10k, Resistor_SMD:R_0603_1608Metric_Pad0.98x0.95mm_HandSolder, F.Cu at (152.0, 92.7)
- added R43: 10k, Resistor_SMD:R_0603_1608Metric_Pad0.98x0.95mm_HandSolder, F.Cu at (153.5, 92.7)
- added R44: 10k, Resistor_SMD:R_0603_1608Metric_Pad0.98x0.95mm_HandSolder, F.Cu at (155.0, 92.7)
- added R45: 47, Resistor_SMD:R_0603_1608Metric_Pad0.98x0.95mm_HandSolder, F.Cu at (153.2, 82.7)
- added R46: 1.2k, Resistor_SMD:R_0603_1608Metric_Pad0.98x0.95mm_HandSolder, F.Cu at (161.1, 93.5)
- added R47: 1.2k, Resistor_SMD:R_0603_1608Metric, F.Cu at (147.2, 106.0)
- added R48: 1.2k, Resistor_SMD:R_0603_1608Metric, F.Cu at (147.2, 107.5)
- added R49: 1.2k, Resistor_SMD:R_0603_1608Metric, F.Cu at (147.2, 109.0)
- added R5: 1.2k, Resistor_SMD:R_0603_1608Metric, F.Cu at (147.2, 149.0)
- added R50: 1.2k, Resistor_SMD:R_0603_1608Metric, F.Cu at (147.2, 84.5)
- added R51: 1.2k, Resistor_SMD:R_0603_1608Metric, F.Cu at (147.2, 86.0)
- added R52: 1.2k, Resistor_SMD:R_0603_1608Metric, F.Cu at (147.2, 87.5)
- added R53: 1.2k, Resistor_SMD:R_0603_1608Metric, F.Cu at (147.2, 88.9)
- added R54: 100k, Resistor_SMD:R_0603_1608Metric, F.Cu at (130.2, 110.4)
- added R55: 330, Resistor_SMD:R_0603_1608Metric, F.Cu at (141.8, 150.3)
- added R56: 330, Resistor_SMD:R_0603_1608Metric, F.Cu at (141.8, 153.4)
- added R57: 330, Resistor_SMD:R_0603_1608Metric, F.Cu at (141.8, 156.6)
- added R58: 4.7k, Resistor_SMD:R_0603_1608Metric, F.Cu at (147.2, 150.5)
- added R59: 4.7k, Resistor_SMD:R_0603_1608Metric, F.Cu at (147.2, 130.5)
- added R6: 1.2k, Resistor_SMD:R_0603_1608Metric, F.Cu at (147.2, 124.5)
- added R60: 4.7k, Resistor_SMD:R_0603_1608Metric, F.Cu at (147.2, 110.5)
- added R61: 4.7k, Resistor_SMD:R_0603_1608Metric, F.Cu at (147.2, 90.4)
- added R7: 1.2k, Resistor_SMD:R_0603_1608Metric, F.Cu at (147.2, 126.0)
- added R8: 1.2k, Resistor_SMD:R_0603_1608Metric, F.Cu at (147.2, 127.5)
- added R9: 1.2k, Resistor_SMD:R_0603_1608Metric, F.Cu at (147.2, 129.0)
- added U1: STM32G0C1KCTxN, Package_QFP:LQFP-32_7x7mm_P0.8mm, F.Cu at (136.4, 96.1)
- added U2: LD1117S33TR_SOT223, Package_TO_SOT_SMD:SOT-223-3_TabPin2, F.Cu at (133.0, 78.0)
- added U3: LM2675M-5.0/NOPB, Package_SO:SOIC-8_3.9x4.9mm_P1.27mm, F.Cu at (148.8, 72.4)
- added U5: MCP2542FDxMF, Package_DFN_QFN:DFN-8-1EP_3x3mm_P0.65mm_EP1.55x2.4mm, F.Cu at (136.9, 124.4)
- moved REF** 45.7 mm to (129.0, 156.0)
- moved REF** 32.1 mm to (161.0, 50.6)
- moved REF** 18.8 mm to (129.0, 64.0)
- moved REF** 7.47 mm to (170.4, 118.5)
Routing:
- net GND: track 0.00 -> 78.3 mm, vias 0 -> 39
- net /SPI1_NSS: track 0.00 -> 77.9 mm, vias 0 -> 4
- net /SPI1_SCK: track 0.00 -> 77.0 mm, vias 0 -> 4
- net /FUSE1_IS: track 0.00 -> 73.5 mm, vias 0 -> 2
- net /LED3: track 0.00 -> 71.1 mm, vias 0 -> 2
- net /LED2: track 0.00 -> 66.6 mm, vias 0 -> 2
- net /LED1: track 0.00 -> 62.1 mm, vias 0 -> 2
- net /SPI1_MOSI: track 0.00 -> 61.0 mm, vias 0 -> 2
- net /LHI_1: track 0.00 -> 55.2 mm, vias 0 -> 2
- net /FUSE2_IS: track 0.00 -> 54.2 mm, vias 0 -> 2
- net /FUSE3_IS: track 0.00 -> 36.6 mm, vias 0 -> 2
- net /LHI_2: track 0.00 -> 35.7 mm, vias 0 -> 2
- net /CAN_RXD: track 0.00 -> 29.8 mm, vias 0 -> 2
- net /CAN_TXD: track 0.00 -> 29.4 mm, vias 0 -> 2
- net /NRST: track 0.00 -> 25.8 mm, vias 0 -> 2
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- added copper zone on F.Cu, net +3.3V
- added copper zone on F.Cu, net +5V
- added copper zone on B.Cu, net +BATT
- added copper zone on F.Cu, net /CAN/CAN_VDD
- added copper zone on F.Cu, net /power/CB
- added copper zone on F.Cu, net /power/SW_L
- added copper zone on F.Cu, net /power/VIN
- added copper zone on F.Cu, net /power/VIN_L
- added copper zone on F.Cu, net /power/VIN_SW_REG
- added copper zone on B.Cu, net GND
- added copper zone on F.Cu, net GND
Other:
- board size 60 x 40 mm -> 55 x 100 mm
- copper layers 2 -> 4
- board text removed: "Template"
- board text removed: "v${REVISION}"

Commit message: Do sprawdzenia
Skończone połączenia
Zrobione przelotki
Parts:
- removed the REF** at (161.0, 50.6)
- added C36: 10n, Capacitor_SMD:C_0603_1608Metric_Pad1.08x0.95mm_HandSolder, B.Cu at (172.5, 152.0)
- moved C43 1.45 mm to (172.6, 132.9)
- moved C41 1.45 mm to (172.6, 125.2)
- moved C33 1.45 mm to (172.6, 140.5)
- moved C34 1.45 mm to (172.6, 144.3)
- moved C35 1.45 mm to (172.6, 148.2)
- moved C42 1.45 mm to (172.6, 129.0)
- moved C44 1.45 mm to (172.6, 136.7)
- moved C58 1.39 mm to (172.6, 88.1)
- moved C59 1.39 mm to (172.6, 91.9)
- moved C60 1.39 mm to (172.6, 95.7)
- moved C49 1.39 mm to (172.6, 99.5)
- moved C50 1.39 mm to (172.6, 103.3)
- moved C51 1.39 mm to (172.6, 107.1)
- moved C52 1.39 mm to (172.6, 111.0)
- moved C57 1.30 mm to (172.6, 84.3)
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Connections:
- C57 pad 1: OUT4_0 -> GND
- C58 pad 1: OUT4_1 -> GND
Routing:
- net +3.3V: track 11.6 -> 185.7 mm, vias 4 -> 2
- net GND: track 78.3 -> 9.01 mm, vias 39 -> 221
- net +5V: track 5.49 -> 55.6 mm, vias 0 -> 2
- net /power/VIN_SW_REG: track 17.9 -> 0.05 mm
- net Net-(U5-VIO): track 1.58 -> 3.12 mm
- net OUT2_0: track 1.20 -> 2.49 mm, vias 1 -> 0
- net OUT2_1: track 1.20 -> 2.48 mm, vias 1 -> 0
- net OUT2_2: track 1.20 -> 2.47 mm, vias 1 -> 0
- net OUT3_3: track 1.20 -> 2.47 mm, vias 1 -> 0
- net OUT3_2: track 1.20 -> 2.47 mm, vias 1 -> 0
- net OUT3_0: track 1.20 -> 2.46 mm, vias 1 -> 0
- net OUT3_1: track 1.20 -> 2.47 mm, vias 1 -> 0
- net OUT2_3: track 1.20 -> 2.46 mm, vias 1 -> 0
- net OUT4_3: track 1.20 -> 2.46 mm, vias 1 -> 0
- net OUT1_2: track 1.20 -> 2.46 mm, vias 1 -> 0
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- added copper zone on In1.Cu, net GND
- added copper zone on In2.Cu, net GND
- added copper zone on F.Cu, net OUT1_0
- added copper zone on F.Cu, net OUT1_1
- added copper zone on F.Cu, net OUT1_2
- added copper zone on F.Cu, net OUT2_0
- added copper zone on F.Cu, net OUT2_1
- added copper zone on F.Cu, net OUT2_2
- added copper zone on F.Cu, net OUT2_3
- added copper zone on F.Cu, net OUT3_0
- added copper zone on F.Cu, net OUT3_1
- added copper zone on F.Cu, net OUT3_2
- added copper zone on F.Cu, net OUT3_3
- added copper zone on F.Cu, net OUT4_2
- added copper zone on F.Cu, net OUT4_3

Commit message: Poprawki
Parts:
- moved D5 8.26 mm to (129.6, 132.8), turned to 90 degrees
- moved R1 6.91 mm to (140.2, 125.7), turned to 180 degrees
- moved JP1 2.51 mm to (137.2, 129.2), turned to 90 degrees
- moved J6 0.85 mm to (128.4, 140.7)
Routing:
- net /CAN/CAN_VDD: track 5.74 -> 2.50 mm
- net CAN_L: track 21.9 -> 24.8 mm, vias 0 -> 2
- net GND: track 9.01 -> 6.77 mm, vias 221 -> 226
- net OUT1_3: track 0.00 -> 1.95 mm
- net OUT4_0: track 0.00 -> 1.95 mm
- net CAN_H: track 22.1 -> 21.2 mm
- net Net-(JP1-B): track 3.15 -> 4.00 mm
- net +5V: track 55.6 -> 54.7 mm
- net OUT4_1: track 0.00 -> 0.65 mm
- net /STM_VCC: track 17.7 -> 17.1 mm

Commit message: Poprawki 3
Parts:
- moved C11 0.23 mm to (138.2, 78.8)
Routing:
- net /power/VIN: track 0.00 -> 4.84 mm
- net GND: vias 226 -> 225
- removed copper zone on F.Cu, net /power/VIN

Commit message: Poprawki 4
Parts:
- moved C11 0.23 mm to (138.2, 79.0)
Routing:
- net /power/VIN: track 4.84 -> 0.00 mm
- net GND: vias 225 -> 226
- added copper zone on F.Cu, net /power/VIN

Commit message: Poprawki 5
Parts:
- moved C11 0.33 mm to (138.2, 78.7)
Routing:
- net /power/VIN: track 0.00 -> 4.84 mm
- net +3.3V: track 185.7 -> 183.7 mm
- removed copper zone on F.Cu, net /power/VIN

Commit message: Poprawki6
Parts:
- removed the D3 at (161.4, 75.8)
- added G***: LOGO, logos:PUTM_LOGO_15mm, B.Cu at (164.9, 64.2)
- added G***: LOGO, Logos:SignatureBox25mm, B.Cu at (143.6, 65.7)
- D3: footprint Diode_SMD:D_SMA -> PESD24VF1BLYL:PESD5V0S1BL315
- moved C57 18.5 mm to (191.0, 85.8)
- moved C58 18.5 mm to (191.0, 87.5)
- moved C36 17.6 mm to (190.1, 152.1)
- moved D3 8.66 mm to (161.5, 74.7), turned to 90 degrees
- moved F1 6.17 mm to (167.4, 70.3), turned to -90 degrees
- moved Dr1 2.69 mm to (162.1, 69.4), turned to 90 degrees
- moved C50 1.18 mm to (172.6, 104.5)
- moved C34 1.15 mm to (172.6, 145.5)
- moved C43 1.14 mm to (172.6, 134.0)
- moved C59 1.12 mm to (172.6, 93.0)
- moved C52 1.05 mm to (172.6, 112.0)
- moved C49 0.99 mm to (172.6, 100.5)
- moved C33 0.98 mm to (172.6, 141.5)
- moved C42 0.96 mm to (172.6, 130.0)
- moved C51 0.86 mm to (172.6, 108.0)
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Routing:
- net OUT2_0: track 2.49 -> 0.00 mm
- net OUT2_1: track 2.48 -> 0.00 mm
- net OUT2_2: track 2.47 -> 0.00 mm
- net OUT3_3: track 2.47 -> 0.00 mm
- net OUT3_2: track 2.47 -> 0.00 mm
- net OUT3_1: track 2.47 -> 0.00 mm
- net OUT2_3: track 2.46 -> 0.00 mm
- net OUT3_0: track 2.46 -> 0.00 mm
- net OUT4_3: track 2.46 -> 0.00 mm
- net OUT1_2: track 2.46 -> 0.00 mm
- net OUT4_2: track 2.46 -> 0.00 mm
- net OUT1_0: track 2.46 -> 0.00 mm
- net OUT1_1: track 2.45 -> 0.00 mm
- net GND: vias 226 -> 223
- added copper zone on B.Cu, net OUT1_0
- added copper zone on B.Cu, net OUT1_1
- added copper zone on B.Cu, net OUT1_2
- added copper zone on B.Cu, net OUT2_0
- added copper zone on B.Cu, net OUT2_1
- added copper zone on B.Cu, net OUT2_2
- added copper zone on B.Cu, net OUT2_3
- added copper zone on B.Cu, net OUT3_0
- added copper zone on B.Cu, net OUT3_1
- added copper zone on B.Cu, net OUT3_2
- added copper zone on B.Cu, net OUT3_3
- added copper zone on B.Cu, net OUT4_2
- added copper zone on B.Cu, net OUT4_3
Other:
- board text added: "Kacper Biadała"
- board text added: "v${REVISION}"
