File: hardware/PDM_1/CAN.kicad_sch (KiCad schematic)
At the start: 9 parts, among them U4 ATA6561-GAQW-N

Commit message: Porządki w folderze
Parts:
- removed U4: ATA6561-GAQW-N, Package_SO:SOIC-8_3.9x4.9mm_P1.27mm, symbol Interface_CAN_LIN:MCP2562-E-MF
- added U5: MCP2542FDxMF, Package_DFN_QFN:DFN-8-1EP_3x3mm_P0.65mm_EP1.55x2.4mm, symbol Interface_CAN_LIN:MCP2542FDxMF
Connections:
- net +3.3V: now also FB2.2; no longer FB2.1
- net CAN_H: now also U5.7 (CANH)
- net CAN_L: now also U5.6 (CANL)
- net CAN_RXD: now also U5.4 (RXD)
- net CAN_TXD: now also U5.1 (TXD)
- net GND: now also U5.2 (VSS), U5.8 (STBY), U5.9 (VSS)
- net CAN_VDD: now reaches C19.1, C8.1, FB3.2
- net CAN_VDD: now also U5.3 (VDD)
- net at C17.1: now also FB2.1, U5.5 (VIO); no longer FB2.2
Other:
- moved on the sheet: C17, C8, FB2, FB3
