File: hardware/PDM_1/battery_connection.kicad_sch (KiCad schematic)
At the start: 3 parts

Commit message: Porządki w folderze
Parts:
- removed C25: C_Small, symbol Device:C_Small
- removed F1: Fuse_Small, symbol Device:Fuse_Small
- D6: now not fitted
Other:
- sheet IC_1 ports: added IS, LHI, OUT0, OUT1, OUT2, OUT3; removed ADC, IN0, IN1, IN2, IN3, out0, out1, out2, out3
- sheet IC_2 ports: added IS, LHI, OUT0, OUT1, OUT2, OUT3; removed ADC, IN0, IN1, IN2, IN3, out0, out1, out2, out3
- sheet IC_3 ports: added IS, LHI, OUT0, OUT1, OUT2, OUT3; removed ADC, IN0, IN1, IN2, IN3, out0, out1, out2, out3
- sheet IC_4 ports: added IS, LHI, OUT0, OUT1, OUT2, OUT3; removed ADC, IN0, IN1, IN2, IN3, out0, out1, out2, out3
- note added: "clk"
- note added: "nss"
- note added: "tvs na schemacie z konektorem"
