File: hardware/PDM_1/IC.kicad_sch (KiCad schematic)
At the start: 19 parts, among them IC1 BTS722204ESAXUMA1

Commit message: Porządki w folderze
Parts:
- added R2, R3, R4, R5: 1.2k, Resistor_SMD:R_0603_1608Metric, symbol Device:R_Small
- added R58: 4.7k, Resistor_SMD:R_0603_1608Metric, symbol Device:R_Small
- C29: renamed from C26; footprint (none) -> Capacitor_SMD:C_0603_1608Metric_Pad1.08x0.95mm_HandSolder
- C30: renamed from C27; footprint (none) -> Capacitor_SMD:C_0603_1608Metric_Pad1.08x0.95mm_HandSolder
- C31: renamed from C28; footprint (none) -> Capacitor_SMD:C_0603_1608Metric_Pad1.08x0.95mm_HandSolder
- C32: renamed from C20; footprint (none) -> Capacitor_SMD:C_0603_1608Metric_Pad1.08x0.95mm_HandSolder
- C33: renamed from C24; footprint (none) -> Capacitor_SMD:C_0603_1608Metric_Pad1.08x0.95mm_HandSolder
- C34: renamed from C23; footprint (none) -> Capacitor_SMD:C_0603_1608Metric_Pad1.08x0.95mm_HandSolder
- C35: renamed from C22; footprint (none) -> Capacitor_SMD:C_0603_1608Metric_Pad1.08x0.95mm_HandSolder
- C36: renamed from C21; footprint (none) -> Capacitor_SMD:C_0603_1608Metric_Pad1.08x0.95mm_HandSolder
- D8: renamed from D7; footprint (none) -> Diode_SMD:D_SMA
- R11: renamed from R10; footprint (none) -> Resistor_SMD:R_0603_1608Metric_Pad0.98x0.95mm_HandSolder
- R12: renamed from R3; footprint (none) -> Resistor_SMD:R_0603_1608Metric_Pad0.98x0.95mm_HandSolder
- R13: renamed from R9; footprint (none) -> Resistor_SMD:R_0603_1608Metric_Pad0.98x0.95mm_HandSolder
- R14: renamed from R5; value 4.7k -> 10k; footprint (none) -> Resistor_SMD:R_0603_1608Metric_Pad0.98x0.95mm_HandSolder
- R15: renamed from R6; value 4.7k -> 10k; footprint (none) -> Resistor_SMD:R_0603_1608Metric_Pad0.98x0.95mm_HandSolder
- R16: renamed from R7; value 4.7k -> 10k; footprint (none) -> Resistor_SMD:R_0603_1608Metric_Pad0.98x0.95mm_HandSolder
- R17: renamed from R8; value 4.7k -> 10k; footprint (none) -> Resistor_SMD:R_0603_1608Metric_Pad0.98x0.95mm_HandSolder
- R18: renamed from R2; footprint (none) -> Resistor_SMD:R_0603_1608Metric_Pad0.98x0.95mm_HandSolder
- R19: renamed from R4; footprint (none) -> Resistor_SMD:R_0603_1608Metric_Pad0.98x0.95mm_HandSolder
- renumbered IC1 to IC2
Connections:
- net 4.7k resistor is gone; now on net IN3: IC2.11 (IN3), R17.2
- net CSN: now also R5.1; no longer IC2.3 (SO), IC2.4 (SI), IC2.5 (SCLK), IC2.6 (CSN)
- net GND: now also R14.1, R15.1, R16.1, R17.1
- net IN0: no longer R14.1
- net IN1: no longer R15.1
- net IN2: no longer R16.1
- net IN3: no longer R17.1
- net VS: now also C30.1, C31.1
- net at C31.2, C32.1, R18.2: now also IC2.1 (GND_1)
- net at IC2.7 (LHI): now also R58.2
- net ADC renamed IS
- net out0 renamed OUT0
- net out1 renamed OUT1
- net out2 renamed OUT2
- net out3 renamed OUT3
- new net: IC2.5 (SCLK), R4.2
- new net: IC2.3 (SO), R2.2
- new net: IC2.6 (CSN), R5.2
- new net: IC2.4 (SI), R3.2
- new net LHI: R58.1
- new net MISO: R2.1
- new net MOSI: R3.1
- new net SCLK: R4.1
Other:
- note added: "gnd czy GPIO?"
- moved on the sheet: IC2

Commit message: Poprawki6
Other:
- note removed: "gnd czy GPIO?"
- note removed: "optional"
Changed lines of the file:
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@@
     (effects (font (size 1.27 1.27)) (justify left bottom))
   )
-  (text "Optional\n" (at 100.33 128.27 0)
-    (effects (font (size 1.27 1.27)) (justify left bottom))
+  (text "Optional\n" (at 104.14 128.27 0)
+    (effects (font (size 0.5 0.5)) (justify left bottom))
   )
   (text "4A max" (at 168.91 81.28 0)
@@
     (effects (font (size 0.6 0.6)) (justify left bottom))
   )
-  (text "optional\n" (at 129.54 50.8 0)
-    (effects (font (size 1.27 1.27)) (justify left bottom))
-  )
   (text "4A max" (at 168.91 88.9 0)
     (effects (font (size 0.6 0.6)) (justify left bottom))
@@
     (effects (font (size 0.6 0.6)) (justify left bottom))
   )
-  (text "gnd czy GPIO?" (at 88.9 90.17 0)
-    (effects (font (size 1.27 1.27)) (justify left bottom))
-  )
   (label "IN2" (at 128.27 93.98 0) (fields_autoplaced)
