File: hardware/PDM_1/connectors.kicad_sch (KiCad schematic)
At the start: 4 parts, among them J2 UPT-08-01-01-L-RA, J5 UPT-02-01-01-X-RA, J6 Conn_01x06, J7 UPT-08-01-01-L-RA

Commit message: Do sprawdzenia
Skończone połączenia
Zrobione przelotki
Connections:
- no-connect marks 1 -> 4
Changed lines of the file:
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@@
   (junction (at 83.82 120.65) (diameter 0) (color 0 0 0 0)
   )
+  (no_connect (at 25.4 114.3))
+  (no_connect (at 34.29 99.06))
   (no_connect (at 176.53 34.29))
+  (no_connect (at 25.4 149.86))
   (wire (pts (xy 106.68 48.26) (xy 106.68 50.8))
     (stroke (width 0) (type default))

Commit message: Poprawki6
Changed lines of the file:
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@@
   (junction (at 83.82 120.65) (diameter 0) (color 0 0 0 0)
   )
-  (no_connect (at 25.4 114.3))
-  (no_connect (at 34.29 99.06))
+  (no_connect (at 25.4 90.17))
+  (no_connect (at 25.4 99.06))
   (no_connect (at 176.53 34.29))
-  (no_connect (at 25.4 149.86))
+  (no_connect (at 25.4 107.95))
   (wire (pts (xy 106.68 48.26) (xy 106.68 50.8))
     (stroke (width 0) (type default))
@@
     )
   )
-  (global_label "OUT4_1" (shape input) (at 25.4 149.86 0) (fields_autoplaced)
-    (effects (font (size 1.27 1.27)) (justify left))
-    (property "Intersheetrefs" "${INTERSHEET_REFS}" (at 35.4004 149.86 0)
+  (global_label "OUT4_1" (shape input) (at 25.4 90.17 0) (fields_autoplaced)
+    (effects (font (size 1.27 1.27)) (justify left))
+    (property "Intersheetrefs" "${INTERSHEET_REFS}" (at 35.4004 90.17 0)
       (effects (font (size 1.27 1.27)) (justify left) hide)
     )
@@
     )
   )
-  (global_label "OUT1_3" (shape input) (at 34.29 99.06 180) (fields_autoplaced)
-    (effects (font (size 1.27 1.27)) (justify right))
-    (property "Intersheetrefs" "${INTERSHEET_REFS}" (at 24.2896 99.06 0)
-      (effects (font (size 1.27 1.27)) (justify right) hide)
+  (global_label "OUT1_3" (shape input) (at 25.4 99.06 0) (fields_autoplaced)
+    (effects (font (size 1.27 1.27)) (justify left))
+    (property "Intersheetrefs" "${INTERSHEET_REFS}" (at 35.4004 99.06 0)
+      (effects (font (size 1.27 1.27)) (justify left) hide)
     )
   )
@@
     )
   )
-  (global_label "OUT4_0" (shape input) (at 25.4 114.3 0) (fields_autoplaced)
-    (effects (font (size 1.27 1.27)) (justify left))
-    (property "Intersheetrefs" "${INTERSHEET_REFS}" (at 35.4004 114.3 0)
-      (effects (font (size 1.27 1.27)) (justify left) hide)
-    )
+  (global_label "OUT4_0" (shape input) (at 25.4 107.95 0) (fields_autoplaced)
+    (effects (font (size 1.27 1.27)) (justify left))
+    (property "Intersheetrefs" "${INTERSHEET_REFS}" (at 35.4004 107.95 0)
+      (effects (font (size 1.27 1.27)) (justify left) hide)
+    )
