File: hardware/PDM_1/power.kicad_sch (KiCad schematic)
At the start: 21 parts, among them U2 LD1117S33TR_SOT223, U3 LM2675M-5

Commit message: Porządki w folderze
Parts:
- removed D12: D_TVS, symbol Device:D_TVS
- removed D2: D_Zener, Diode_SMD:D_SOD-123, symbol Device:D_Zener
- removed D3: D_Schottky_Small, Diode_SMD:D_SOD-123, symbol Device:D_Schottky_Small
- removed L2: 47u, Inductor_SMD:L_6.2x5.9_H5, symbol Device:L_Small
- added D3: PESD24VF1BLYL, Diode_SMD:D_SMA, symbol Device:D_TVS
- added F1: 2920L050_72DR, 2920l:FUSC7451X125N, symbol Device:Fuse_Small
- added L4: 47u, Inductor_SMD:L_6.3x6.3_H3, symbol Device:L_Small
- C14: footprint Capacitor_Tantalum_SMD:CP_EIA-7343-31_Kemet-D -> Capacitor_SMD:CP_Elec_6.3x5.4
- Dr1: renamed from D1; value 1N5822 -> SS34ALH; footprint Diode_THT:D_DO-201AD_P15.24mm_Horizontal -> Diode_SMD:D_SMA
- L1: mouser (none) -> https://www.mouser.pl/ProductDetail/ABRACON/ASMPL-0603-R33M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
- U3: value LM2675M-5 -> LM2675M-5.0/NOPB
Connections:
- net +5V: now also C10.1, U2.3 (VI), L4.2
- net GND: now also D3.1 (A1)
- net VIN_L: now also D3.2 (A2)
- net CB: now reaches C12.1, U3.1 (CB)
- net SW_L: now reaches C12.2, D4.1 (K), U3.8 (VSW)
- net SW_L: now also L4.1
- net +24V renamed VIN
- net VIN: now also F1.1
- new net +BATT: F1.2
Other:
- note added: "footprint? chyba git"
- note removed: "100n 1u"
- note removed: "footprint?"

Commit message: Poprawki6
Parts:
- D3: footprint Diode_SMD:D_SMA -> PESD24VF1BLYL:PESD5V0S1BL315
Changed lines of the file:
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@@
     (effects (font (size 1.27 1.27)) (justify left bottom))
   )
-  (text "5v to 3.3V" (at 147.955 118.11 0)
+  (text "5v to 3.3V" (at 149.86 119.38 0)
     (effects (font (size 1.27 1.27)) (justify left bottom))
   )
@@
       (effects (font (size 1.27 1.27)) (justify left))
     )
-    (property "Footprint" "Diode_SMD:D_SMA" (at 76.2 87.63 0)
-      (effects (font (size 1.27 1.27)) hide)
-    )
+    (property "Footprint" "PESD24VF1BLYL:PESD5V0S1BL315" (at 76.2 87.63 0)
+      (effects (font (size 1.27 1.27)) hide)
+    )

Commit message: Koniec
Parts:
- D3: value PESD24VF1BLYL -> SMAJ24CA-13-F; footprint PESD24VF1BLYL:PESD5V0S1BL315 -> Diode_SMD:D_SMA; Manufacturer_Part_Number PESD24VF1BLYL -> SMAJ24CA-13-F; Mouser Part Number 771-PESD24VF1BLYL -> 621-SMAJ24CA-13-F; Mouser Price/Stock https://www.mouser.co.uk/ProductDetail/Nexperia/PESD24VF1BL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 -> https://www.mouser.pl/ProductDetail/Diodes-Incorporated/SMA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; description PESD24VF1BL - Ultra low capacitance bidirectional ESD prote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 -> (none)
Other:
- note removed: "footprint? chyba git"
Changed lines of the file:
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@@
     (stroke (width 0) (type default))
-  )
-  (text "footprint? chyba git" (at 50.8 92.71 0)
-    (effects (font (size 1.27 1.27)) (justify left bottom))
   )
   (text "5v to 3.3V" (at 149.86 119.38 0)
@@
       (effects (font (size 1.27 1.27)) (justify left))
     )
-    (property "Value" "PESD24VF1BLYL" (at 73.66 88.9 90)
-      (effects (font (size 1.27 1.27)) (justify left))
-    )
-    (property "Footprint" "PESD24VF1BLYL:PESD5V0S1BL315" (at 76.2 87.63 0)
-      (effects (font (size 1.27 1.27)) hide)
-    )
-    (property "Datasheet" "https://assets.nexperia.com/documents/data-sheet/PESD24VF1BL.pdf" (at 76.2 87.63 0)
-      (effects (font (size 1.27 1.27)) hide)
-    )
-    (property "description" "PESD24VF1BL - Ultra low capacitance bidirectional ESD protection diode" (at 76.2 87.63 90)
-      (effects (font (size 1.27 1.27)) hide)
-    )
-    (property "Mouser Part Number" "771-PESD24VF1BLYL" (at 76.2 87.63 90)
+    (property "Value" "SMAJ24CA-13-F" (at 73.66 88.9 90)
+      (effects (font (size 1.27 1.27)) (justify left))
+    )
+    (property "Footprint" "Diode_SMD:D_SMA" (at 76.2 87.63 0)
+      (effects (font (size 1.27 1.27)) hide)
+    )
+    (property "Datasheet" "https://www.mouser.pl/datasheet/2/115/DIOD_S_A0011538071_1-2543697.pdf" (at 76.2 87.63 0)
+      (effects (font (size 1.27 1.27)) hide)
+    )
+    (property "Mouser Part Number" "621-SMAJ24CA-13-F" (at 76.2 87.63 90)
       (effects (font (size 1.27 1.27)) (justify left bottom) hide)
     )
-    (property "Mouser Price/Stock" "https://www.mouser.co.uk/ProductDetail/Nexperia/PESD24VF1BLYL?qs=M%2FOdCRO8QQ2u4QQQVkgemw%3D%3D" (at 76.2 87.63 90)
+    (property "Mouser Price/Stock" "https://www.mouser.pl/ProductDetail/Diodes-Incorporated/SMAJ24CA-13-F?qs=gaDBXWSqsDA5MVRJAApKgw%3D%3D" (at 76.2 87.63 90)
       (effects (font (size 1.27 1.27)) (justify left bottom) hide)
     )
-    (property "Manufacturer_Part_Number" "PESD24VF1BLYL" (at 76.2 87.63 90)
+    (property "Manufacturer_Part_Number" "SMAJ24CA-13-F" (at 76.2 87.63 90)
       (effects (font (size 1.27 1.27)) (justify left bottom) hide)
     )
