File: PUTM_EV_PDM-main2/PUTM_EV_PDM-main/hardware/PDM_1/LED.kicad_sch (KiCad schematic)
At the start: 6 parts

Commit message: małe zmiany
dodano złącza
zmieniono parę footprintów
Parts:
- renumbered D5 to D1, D6 to D2, R1 to R55, R2 to R56, R3 to R57
Changed lines of the file:
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@@
   (symbol (lib_id "Device:R") (at 72.39 62.23 90) (unit 1)
     (in_bom yes) (on_board yes) (dnp no) (fields_autoplaced)
-    (property "Reference" "R2" (at 72.39 55.88 90)
+    (property "Reference" "R56" (at 72.39 55.88 90)
       (effects (font (size 1.27 1.27)))
     )
@@
   (symbol (lib_id "Device:R") (at 72.39 50.8 90) (unit 1)
     (in_bom yes) (on_board yes) (dnp no) (fields_autoplaced)
-    (property "Reference" "R1" (at 72.39 44.45 90)
+    (property "Reference" "R55" (at 72.39 44.45 90)
       (effects (font (size 1.27 1.27)))
     )
@@
   (symbol (lib_id "Device:LED") (at 85.09 50.8 180) (unit 1)
     (in_bom yes) (on_board yes) (dnp no) (fields_autoplaced)
-    (property "Reference" "D5" (at 86.6775 43.18 0)
+    (property "Reference" "D1" (at 86.6775 43.18 0)
       (effects (font (size 1.27 1.27)))
     )
@@
   (symbol (lib_id "power:+3.3V") (at 55.88 62.23 0) (unit 1)
     (in_bom yes) (on_board yes) (dnp no) (fields_autoplaced)
-    (property "Reference" "#PWR012" (at 55.88 66.04 0)
+    (property "Reference" "#PWR051" (at 55.88 66.04 0)
       (effects (font (size 1.27 1.27)) hide)
     )
@@
   (symbol (lib_id "Device:LED") (at 85.09 62.23 180) (unit 1)
     (in_bom yes) (on_board yes) (dnp no) (fields_autoplaced)
-    (property "Reference" "D6" (at 86.6775 54.61 0)
+    (property "Reference" "D2" (at 86.6775 54.61 0)
       (effects (font (size 1.27 1.27)))
     )
@@
   (symbol (lib_id "Device:R") (at 72.39 73.66 90) (unit 1)
     (in_bom yes) (on_board yes) (dnp no) (fields_autoplaced)
-    (property "Reference" "R3" (at 72.39 67.31 90)
+    (property "Reference" "R57" (at 72.39 67.31 90)
       (effects (font (size 1.27 1.27)))
     )
