File: PUTM_EV_PDM-main2/PUTM_EV_PDM-main/hardware/PDM_1/_autosave-power.kicad_sch (KiCad schematic)
At the start: 20 parts, among them U2 LD1117S33TR_SOT223, U3 LM2675M-5

Commit message: piny na płytce
Dodano ułożenie pinów na płytce
Parts:
- Dr1: value 1N5822 -> SS34ALH
Changed lines of the file:
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@@
       (effects (font (size 1.27 1.27)) (justify right))
     )
-    (property "Value" "1N5822" (at 78.74 70.1675 90)
+    (property "Value" "SS34ALH" (at 78.74 70.1675 90)
       (effects (font (size 1.27 1.27)) (justify right))
     )
