File: PUTM_EV_PDM-main2/PUTM_EV_PDM-main/hardware/PDM_1/_autosave-power.kicad_sch (KiCad schematic)
At the start: 20 parts, among them U2 LD1117S33TR_SOT223, U3 LM2675M-5

Commit message: Połączenia w grupach
Parts:
- U3: value LM2675M-5 -> LM2675M-5.0/NOPB
Connections:
- net CB: now reaches C12.1, U3.1 (CB)
- net VIN: now reaches Dr1.2 (A), F1.1
Changed lines of the file:
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@@
     (effects (font (size 1.27 1.27)) (justify left bottom))
   )
+  (label "VIN" (at 76.2 63.5 180) (fields_autoplaced)
+    (effects (font (size 0.5 0.5)) (justify right bottom))
+  )
+  (label "CB" (at 170.18 82.55 0) (fields_autoplaced)
+    (effects (font (size 0.5 0.5)) (justify left bottom))
+  )
   (label "VIN_SW_REG" (at 135.89 77.47 180) (fields_autoplaced)
+    (effects (font (size 0.5 0.5)) (justify right bottom))
+  )
+  (label "VIN_L" (at 76.2 80.01 180) (fields_autoplaced)
     (effects (font (size 0.5 0.5)) (justify right bottom))
   )
@@
       (effects (font (size 1.27 1.27)))
     )
-    (property "Value" "LM2675M-5" (at 156.21 72.39 0)
+    (property "Value" "LM2675M-5.0/NOPB" (at 156.21 72.39 0)
       (effects (font (size 1.27 1.27)))
     )
