File: PUTM_EV_PDM-main2/PUTM_EV_PDM-main/hardware/PDM_1/_autosave-PDM_1.kicad_sch (KiCad schematic)
At the start: 8 parts, among them J1 FTSH-107-01-L-DV-K-A, U1 STM32G0C1KCTxN

Commit message: Nowe ułożenie na płytce
Ułożenie komponentów na płytce
Dodane połączenie +24V
Connections:
- net LED1: now also U1.19 (PA9/UCPD1_DBCC1); no longer U1.18 (PA8)
- net LED2: now also U1.18 (PA8); no longer U1.19 (PA9/UCPD1_DBCC1)
- net STM_VCC: now reaches C1.1, C2.1, C3.1, C4.1, FB1.2, U1.20 (VDDIO2), U1.4 (VDD)
Changed lines of the file:
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@@
     (effects (font (size 1.27 1.27)) (justify left bottom))
   )
-  (label "LED2" (at 260.35 69.85 0) (fields_autoplaced)
+  (label "LED2" (at 260.35 67.31 0) (fields_autoplaced)
     (effects (font (size 1.27 1.27)) (justify left bottom))
   )
@@
     (effects (font (size 1.27 1.27)) (justify left bottom))
   )
-  (label "LED1" (at 260.35 67.31 0) (fields_autoplaced)
+  (label "LED1" (at 260.35 69.85 0) (fields_autoplaced)
     (effects (font (size 1.27 1.27)) (justify left bottom))
   )
@@
     (effects (font (size 1.27 1.27)) (justify left bottom))
   )
+  (label "STM_VCC" (at 191.77 26.67 0) (fields_autoplaced)
+    (effects (font (size 1.27 1.27)) (justify left bottom))
+  )
