File: PUTM_EV_PDM-main2/PUTM_EV_PDM-main/hardware/PDM_1/PDM_1.kicad_sch (KiCad schematic)
At the start: 8 parts, among them J1 FTSH-107-01-L-DV-K-A, U1 STM32G0C1KCTxN

Commit message: Koniec połączeń sygnałów
Wszystkie sygnały z stm poprowadzone
Zmienione ułożenie połączeń do złącz
Connections:
- net +3V3 is gone; now on net +3.3V: R1.2
- net CAN_RXD: no longer U1.26 (PD0)
- net CAN_TXD: no longer U1.27 (PD1)
- net LED1: now also U1.19 (PA9/UCPD1_DBCC1); no longer U1.18 (PA8)
- net LED2: now also U1.18 (PA8); no longer U1.19 (PA9/UCPD1_DBCC1)
- no-connect marks 10 -> 12
Other:
- note added: "?"
- note added: "can_rxd"
- note added: "can_txd ???"
Changed lines of the file:
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@@
   (junction (at 201.93 26.67) (diameter 0) (color 0 0 0 0)
   )
+  (junction (at 241.3 99.06) (diameter 0) (color 0 0 0 0)
+  )
   (junction (at 189.23 26.67) (diameter 0) (color 0 0 0 0)
   )
   (junction (at 39.37 157.48) (diameter 0) (color 0 0 0 0)
   )
+  (junction (at 233.68 26.67) (diameter 0) (color 0 0 0 0)
+  )
   (junction (at 241.3 39.37) (diameter 0) (color 0 0 0 0)
   )
@@
   (junction (at 34.29 162.56) (diameter 0) (color 0 0 0 0)
   )
+  (no_connect (at 219.71 52.07))
+  (no_connect (at 219.71 54.61))
   (no_connect (at 54.61 149.86))
   (no_connect (at 220.98 67.31))
@@
     (stroke (width 0) (type default))
   )
-  (wire (pts (xy 227.33 26.67) (xy 241.3 26.67))
+  (wire (pts (xy 227.33 26.67) (xy 233.68 26.67))
     (stroke (width 0) (type default))
   )
@@
     (stroke (width 0) (type default))
   )
-  (wire (pts (xy 241.3 95.25) (xy 241.3 102.87))
+  (wire (pts (xy 233.68 26.67) (xy 241.3 26.67))
+    (stroke (width 0) (type default))
+  )
+  (wire (pts (xy 241.3 95.25) (xy 241.3 99.06))
     (stroke (width 0) (type default))
   )
@@
     (stroke (width 0) (type default))
   )
-  (wire (pts (xy 160.02 63.5) (xy 160.02 62.23))
-    (stroke (width 0) (type default))
-  )
   (wire (pts (xy 214.63 26.67) (xy 214.63 30.48))
     (stroke (width 0) (type default))
@@
     (stroke (width 0) (type default))
   )
+  (wire (pts (xy 241.3 99.06) (xy 241.3 102.87))
+    (stroke (width 0) (type default))
+  )
   (wire (pts (xy 214.63 35.56) (xy 214.63 39.37))
     (stroke (width 0) (type default))
@@
     (fill (type none))
   )
+  (text "can_txd\n???" (at 203.2 55.88 0)
+    (effects (font (size 1.27 1.27)) (justify left bottom))
+  )
+  (text "?" (at 176.53 31.75 0)
+    (effects (font (size 1.27 1.27)) (justify left bottom))
+  )
+  (text "can_rxd" (at 203.2 52.07 0)
+    (effects (font (size 1.27 1.27)) (justify left bottom))
+  )
   (text "złącza\n" (at 26.67 139.7 0)
     (effects (font (size 1.27 1.27)) (justify left bottom))
@@
     (effects (font (size 1.27 1.27)) (justify left bottom))
   )
-  (label "CAN_TXD" (at 219.71 54.61 180) (fields_autoplaced)
-    (effects (font (size 1.27 1.27)) (justify right bottom))
-  )
   (label "LED3" (at 219.71 87.63 180) (fields_autoplaced)
     (effects (font (size 1.27 1.27)) (justify right bottom))
@@
     (effects (font (size 1.27 1.27)) (justify left bottom))
   )
-  (label "LED2" (at 260.35 69.85 0) (fields_autoplaced)
+  (label "LED2" (at 260.35 67.31 0) (fields_autoplaced)
     (effects (font (size 1.27 1.27)) (justify left bottom))
   )
@@
     (effects (font (size 1.27 1.27)) (justify left bottom))
   )
-  (label "LED1" (at 260.35 67.31 0) (fields_autoplaced)
+  (label "LED1" (at 260.35 69.85 0) (fields_autoplaced)
     (effects (font (size 1.27 1.27)) (justify left bottom))
   )
@@
   (label "LED2" (at 41.91 114.3 0) (fields_autoplaced)
     (effects (font (size 1.27 1.27)) (justify left bottom))
-  )
-  (label "CAN_RXD" (at 219.71 52.07 180) (fields_autoplaced)
-    (effects (font (size 1.27 1.27)) (justify right bottom))
   )
   (global_label "CAN_L" (shape input) (at 64.77 31.75 0) (fields_autoplaced)
@@
     )
   )
+  (symbol (lib_id "power:PWR_FLAG") (at 241.3 99.06 90) (unit 1)
+    (in_bom yes) (on_board yes) (dnp no) (fields_autoplaced)
+    (property "Reference" "#FLG05" (at 239.395 99.06 0)
+      (effects (font (size 1.27 1.27)) hide)
+    )
+    (property "Value" "PWR_FLAG" (at 237.49 99.06 90)
+      (effects (font (size 1.27 1.27)) (justify left))
+    )
+    (property "Footprint" "" (at 241.3 99.06 0)
+      (effects (font (size 1.27 1.27)) hide)
+    )
+    (property "Datasheet" "~" (at 241.3 99.06 0)
+      (effects (font (size 1.27 1.27)) hide)
+    )
+    (pin "1")
+    (instances
+      (project "PDM_1"
+        (path "/b652b05a-4e3d-4ad1-b032-18886abe7d45"
+          (reference "#FLG05") (unit 1)
+        )
+      )
+    )
+  )
   (symbol (lib_id "Device:R_Small") (at 166.37 63.5 270) (unit 1)
     (in_bom yes) (on_board yes) (dnp no)
@@
         (path "/d7434f1a-7415-4eaa-a71b-b9580d7b34f2"
           (reference "C10") (unit 1)
+        )
+      )
+    )
+  )
+  (symbol (lib_id "power:+3.3V") (at 160.02 63.5 90) (unit 1)
+    (in_bom yes) (on_board yes) (dnp no) (fields_autoplaced)
+    (property "Reference" "#PWR053" (at 163.83 63.5 0)
+      (effects (font (size 1.27 1.27)) hide)
+    )
+    (property "Value" "+3.3V" (at 156.21 63.5 90)
+      (effects (font (size 1.27 1.27)) (justify left))
+    )
+    (property "Footprint" "" (at 160.02 63.5 0)
+      (effects (font (size 1.27 1.27)) hide)
+    )
+    (property "Datasheet" "" (at 160.02 63.5 0)
+      (effects (font (size 1.27 1.27)) hide)
+    )
+    (pin "1")
+    (instances
+      (project "PDM_1"
+        (path "/b652b05a-4e3d-4ad1-b032-18886abe7d45"
+          (reference "#PWR053") (unit 1)
         )
       )
@@
     )
   )
+  (symbol (lib_id "power:PWR_FLAG") (at 233.68 26.67 0) (unit 1)
+    (in_bom yes) (on_board yes) (dnp no) (fields_autoplaced)
+    (property "Reference" "#FLG06" (at 233.68 24.765 0)
+      (effects (font (size 1.27 1.27)) hide)
+    )
+    (property "Value" "PWR_FLAG" (at 233.68 21.59 0)
+      (effects (font (size 1.27 1.27)))
+    )
+    (property "Footprint" "" (at 233.68 26.67 0)
+      (effects (font (size 1.27 1.27)) hide)
+    )
+    (property "Datasheet" "~" (at 233.68 26.67 0)
+      (effects (font (size 1.27 1.27)) hide)
+    )
+    (pin "1")
+    (instances
+      (project "PDM_1"
+        (path "/b652b05a-4e3d-4ad1-b032-18886abe7d45"
+          (reference "#FLG06") (unit 1)
+        )
+      )
+    )
+  )
   (symbol (lib_id "power:GND") (at 241.3 102.87 0) (unit 1)
     (in_bom yes) (on_board yes) (dnp no) (fields_autoplaced)
@@
         )
       )
-    )
-  )
-  (symbol (lib_id "BMS_LV_2022-rescue:+3.3V-power") (at 160.02 62.23 0) (unit 1)
-    (in_bom yes) (on_board yes) (dnp no)
-    (property "Reference" "#PWR02" (at 160.02 66.04 0)
-      (effects (font (size 1.27 1.27)) hide)
-    )
-    (property "Value" "+3.3V" (at 160.401 57.8358 0)
-      (effects (font (size 1.27 1.27)))
-    )
-    (property "Footprint" "" (at 160.02 62.23 0)
-      (effects (font (size 1.27 1.27)) hide)
-    )
-    (property "Datasheet" "" (at 160.02 62.23 0)
-      (effects (font (size 1.27 1.27)) hide)
-    )
-    (pin "1")
-    (instances
-      (project "BMS_LV_2022"
-        (path "/9e2228b4-33a3-45e8-b8af-05631e0178ab"
-          (reference "#PWR02") (unit 1)
-        )
-      )
-      (project "PDM_1"
-        (path "/b652b05a-4e3d-4ad1-b032-18886abe7d45"
-          (reference "#PWR050") (unit 1)
-        )
-      )
